File: PeekaBot V1!!/CAD/PCB/peekabot_pcb_v1/peekabot_pcb_v1.kicad_sch (KiCad schematic)
At the start: 7 parts, among them J1 esp32camright, J2 esp32camleft, J3 USB_B_Micro, SW1 SW_Push

Commit message: started working on the schematics of the pcb
Parts:
- added C3, C4: 22uF, Capacitor_SMD:C_0805_2012Metric, symbol Device:C
- added C5, C6, C7: 10uF, Capacitor_SMD:C_0805_2012Metric, symbol Device:C
- added C8: 110uF, Capacitor_SMD:C_0805_2012Metric, symbol Device:C
- added C9: 220uF, Capacitor_SMD:C_0805_2012Metric, symbol Device:C
- added D1, D2, D3: LED, LED_SMD:LED_0805_2012Metric_Pad1.15x1.40mm_HandSolder, symbol Device:LED
- added J4: Battery Socket, Connector_JST:JST_EH_S2B-EH_1x02_P2.50mm_Horizontal, symbol Connector:Conn_01x02_Socket
- added L1: 1uH, Inductor_SMD:L_7.3x7.3_H3.5, symbol Device:L
- added R2: R, Resistor_SMD:R_0805_2012Metric, symbol Device:R
- added R3: 20R, Resistor_SMD:R_0805_2012Metric, symbol Device:R
- added R4: 10kR, Resistor_SMD:R_0805_2012Metric, symbol Device:R
- added R5: 2R, Resistor_SMD:R_0805_2012Metric, symbol Device:R
- added SW2: SW_Push, Button_Switch_SMD:SW_Push_1P1T_NO_CK_KMR2, symbol Switch:SW_Push
- added U1: IP5306, IP5306:SOP127P600X165-9N, symbol IP5306:IP5306
- C1: value 100uf -> 10uF; footprint (none) -> Capacitor_SMD:C_0805_2012Metric
- C2: value 0.1uf -> 22uF; footprint (none) -> Capacitor_SMD:C_0805_2012Metric
- J1, J2: footprint (none) -> Connector_PinSocket_2.54mm:PinSocket_1x08_P2.54mm_Vertical
- J3: footprint (none) -> Connector_USB:USB_Micro-B_Molex-105017-0001
- R1: footprint (none) -> Resistor_SMD:R_0805_2012Metric
- SW1: footprint (none) -> Button_Switch_SMD:SW_Push_1P1T_NO_CK_KMR2
Connections:
- net 5V: now also C2.1, C3.1, C4.1, C8.1, C9.1, U1.8 (VOUT)
- net GND: now also C1.2, C2.2, C3.2, C4.2, C5.2, C6.2, C7.2, C8.2, C9.2, D1.1 (K), D2.1 (K), D3.1 (K), J4.2 (Pin_2), SW2.2, U1.9 (POWERPAD); no longer C1.1, C2.1
- net VCC: no longer C1.2, C2.2, J3.1 (VBUS)
- new net: C1.1, J3.1 (VBUS), R2.1, U1.1 (VIN)
- new net: D2.2 (A), U1.2 (LED1)
- new net: D3.2 (A), U1.4 (LED3)
- new net: R3.1, R4.1, U1.5 (KEY)
- new net: L1.1, U1.7 (SW)
- new net: C5.1, R2.2
- new net: R4.2, SW2.1
- new net: D1.2 (A), R3.2
- new net: C7.1, R5.2
- new net BAT: C6.1, J4.1 (Pin_1), L1.2, R5.1, U1.3 (LED2), U1.6 (BAT)
